File: pcb/adc_fpga/adc_fpga.kicad_sch (KiCad schematic)
At the start: 44 parts, among them J1 RF_IN, J3 AUX I/O, J5 AUX I/O, Q1 BSS138, Q2 BSS138, U1 MAX4230AXK, U2 CMOD S7, U3 ADC14L020CIVY/NOPB, U4 TLV76133DCY

Commit message: LCD kind of working
Other:
- note added: "Audio anti-aliasing"
Changed lines of the file:
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@@
 	(wire
 		(pts
-			(xy 224.79 77.47) (xy 233.68 77.47)
+			(xy 218.44 77.47) (xy 233.68 77.47)
 		)
 		(stroke
@@
 	(wire
 		(pts
-			(xy 218.44 49.53) (xy 224.79 49.53)
-		)
-		(stroke
-			(width 0)
-			(type default)
-		)
-	)
-	(wire
-		(pts
 			(xy 77.47 170.18) (xy 77.47 172.72)
 		)
@@
 	(wire
 		(pts
-			(xy 224.79 49.53) (xy 224.79 77.47)
+			(xy 218.44 45.72) (xy 218.44 77.47)
 		)
 		(stroke
@@
 		(pts
 			(xy 78.74 35.56) (xy 78.74 36.83)
-		)
-		(stroke
-			(width 0)
-			(type default)
-		)
-	)
-	(wire
-		(pts
-			(xy 218.44 45.72) (xy 218.44 49.53)
 		)
 		(stroke
@@
 		(effects
 			(font
+				(size 1.27 1.27)
+			)
+		)
+	)
+	(text "Audio anti-aliasing"
+		(exclude_from_sim no)
+		(at 234.442 21.082 0)
+		(effects
+			(font
