File: pcb/filter_pcb/filter/filter.kicad_pcb (KiCad board)
At the start: 2 copper layers, 50.4 x 37.2 mm, 17 parts, among them J1 IN, J2 OUT

Commit message: WIP
Parts:
- removed the REF** at (135.1, 123.2)
- added REF**: MountingHole_2.2mm_M2_DIN965_Pad, MountingHole:MountingHole_2.2mm_M2_DIN965_Pad, F.Cu at (187.7, 104.1)
- REF** (x3): value MountingHole_2.2mm_M2 -> MountingHole_2.2mm_M2_DIN965_Pad; footprint MountingHole:MountingHole_2.2mm_M2 -> MountingHole:MountingHole_2.2mm_M2_DIN965_Pad
- moved REF** 52.6 mm to (187.7, 91.7)
- moved J2 51.6 mm to (181.1, 98.6)
- moved L5 45.9 mm to (168.9, 98.3)
- moved L3 43.1 mm to (154.7, 98.3)
- moved C5 37.6 mm to (164.3, 96.5), turned to 90 degrees
- moved C4 35.1 mm to (150.1, 96.8), turned to 90 degrees
- moved L2 28.8 mm to (126.2, 98.6)
- moved C3 27.0 mm to (135.9, 97.0), turned to 90 degrees
- moved L4 24.5 mm to (140.5, 98.6)
- moved C1 22.9 mm to (107.4, 94.3), turned to -90 degrees
- moved C2 21.4 mm to (121.7, 94.5), turned to -90 degrees
- moved REF** 19.3 mm to (87.6, 104.1)
- moved R1 12.6 mm to (103.1, 101.9), turned to 90 degrees
- moved L1 7.78 mm to (112.0, 98.3)
- moved REF** 2.79 mm to (87.6, 91.7)
- renumbered C2 to C1, C3 to C2, C1 to C3, C5 to C4, C4 to C5, L5 to L3, L3 to L4, L4 to L5
Connections:
- REF** pad : (no net) -> GND
Routing:
- net Net-(C3-Pad2): track 10.4 -> 5.21 mm
- net Net-(C5-Pad2): track 10.3 -> 6.25 mm
- net Net-(J1-In): track 11.1 -> 8.61 mm
- net Net-(C1-Pad2): track 20.5 -> 22.9 mm
- net Net-(J2-In): track 25.9 -> 24.1 mm
- net Net-(C2-Pad1): track 23.0 -> 21.8 mm
- net GND: vias 68 -> 107
- net (no net): vias 1 -> 0
Other:
- board size 50.4 x 37.2 mm -> 106 x 18.4 mm
