File: pcb/filter_pcb/filter/filter.kicad_sch (KiCad schematic)
At the start: 13 parts, among them J1 IN, J2 OUT

Commit message: LCD kind of working
Parts:
- renumbered C2 to C1, C3 to C2, C1 to C3, C5 to C4, C4 to C5, L5 to L3, L3 to L4, L4 to L5
Changed lines of the file:
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@@
 		(dnp no)
 		(fields_autoplaced yes)
-		(property "Reference" "C1"
+		(property "Reference" "C3"
 			(at 110.49 80.0099 0)
 			(effects
@@
 			(project "filter"
 				(path "/816b9c7a-dde1-46d5-96e5-a392ccbb4253"
-					(reference "C1")
+					(reference "C3")
 					(unit 1)
 				)
@@
 		(dnp no)
 		(fields_autoplaced yes)
-		(property "Reference" "C3"
+		(property "Reference" "C2"
 			(at 87.63 66.04 90)
 			(effects
@@
 			(project "filter"
 				(path "/816b9c7a-dde1-46d5-96e5-a392ccbb4253"
-					(reference "C3")
+					(reference "C2")
 					(unit 1)
 				)
@@
 		(dnp no)
 		(fields_autoplaced yes)
-		(property "Reference" "C5"
+		(property "Reference" "C4"
 			(at 129.54 66.04 90)
 			(effects
@@
 			(project "filter"
 				(path "/816b9c7a-dde1-46d5-96e5-a392ccbb4253"
-					(reference "C5")
+					(reference "C4")
 					(unit 1)
 				)
@@
 		(dnp no)
 		(fields_autoplaced yes)
-		(property "Reference" "L3"
+		(property "Reference" "L4"
 			(at 120.65 80.0099 0)
 			(effects
@@
 			(project "filter"
 				(path "/816b9c7a-dde1-46d5-96e5-a392ccbb4253"
-					(reference "L3")
+					(reference "L4")
 					(unit 1)
 				)
@@
 		(dnp no)
 		(fields_autoplaced yes)
-		(property "Reference" "C2"
+		(property "Reference" "C1"
 			(at 67.31 80.0099 0)
 			(effects
@@
 			(project "filter"
 				(path "/816b9c7a-dde1-46d5-96e5-a392ccbb4253"
-					(reference "C2")
+					(reference "C1")
 					(unit 1)
 				)
@@
 		(dnp no)
 		(fields_autoplaced yes)
-		(property "Reference" "L5"
+		(property "Reference" "L3"
 			(at 143.51 68.58 90)
 			(effects
@@
 			(project "filter"
 				(path "/816b9c7a-dde1-46d5-96e5-a392ccbb4253"
-					(reference "L5")
+					(reference "L3")
 					(unit 1)
 				)
@@
 		(dnp no)
 		(fields_autoplaced yes)
-		(property "Reference" "C4"
+		(property "Reference" "C5"
 			(at 156.21 80.0099 0)
 			(effects
@@
 			(project "filter"
 				(path "/816b9c7a-dde1-46d5-96e5-a392ccbb4253"
-					(reference "C4")
+					(reference "C5")
 					(unit 1)
 				)
@@
 		(dnp no)
 		(fields_autoplaced yes)
-		(property "Reference" "L4"
+		(property "Reference" "L5"
 			(at 168.91 80.0099 0)
 			(effects
@@
 			(project "filter"
 				(path "/816b9c7a-dde1-46d5-96e5-a392ccbb4253"
-					(reference "L4")
-					(unit 1)
-				)
+					(reference "L5")
+					(unit 1)
+				)
